Commit message: [Rolling] Release v0.6.0 (#15)
Update the CRCOpen ROS 2 driver for ROS 2 Rolling.

- Add support for up to ten axes.
- Add generic linear-axis position and velocity support.
- Add mock hardware support.
- Replace Python launch files with XML launch files.
- Update controller configuration, visual meshes, Docker configuration, and documentation.
- Set package versions to 0.6.0 and add the changelog.

File: comau_robots/comau_nj_130_2_6_description/urdf/nj_130_2_6.ros2_control.xacro (robot description, xacro)
@@ -1,89 +1,108 @@
 <?xml version="1.0"?>
 <robot xmlns:xacro="http://www.ros.org/wiki/xacro">
-  <xacro:macro name="all_command_and_state_interfaces">
-    <command_interface name="position"/>
-    <command_interface name="position_direct"/>
-    <command_interface name="velocity"/>
-    <command_interface name="acceleration"/>
-    <command_interface name="current"/>
-    <command_interface name="effort"/>
-    <state_interface name="position"/>
-    <state_interface name="velocity"/>
-    <state_interface name="acceleration"/>
-    <state_interface name="current"/>
-    <state_interface name="effort"/>
+  <xacro:include filename="$(find comau_nj_130_2_6_description)/urdf/helper_macros.urdf.xacro" />
+  <xacro:macro name="comau_nj_130_2_6_ros2_control" params="hardware:=crcopen">
+    <ros2_control name="comau_nj_130_2_6" type="system">
+      <hardware>
+        <xacro:if value="${hardware == 'mock'}">
+          <plugin>mock_components/GenericSystem</plugin>
+        </xacro:if>
+        <xacro:if value="${hardware == 'crcopen'}">
+          <plugin>crcopen_hardware/CRCOpenHardware</plugin>
+          <!-- Set IP addresses -->
+          <param name="lpc_addr">169.254.100.2</param>
+          <param name="crc_addr">169.254.100.1</param>
+          <!-- Set payload parameters -->
+          <param name="payload_mass">0.0</param>
+          <param name="payload_cog_x">0.0</param>
+          <param name="payload_cog_y">0.0</param>
+          <param name="payload_cog_z">0.0</param>
+          <param name="payload_inertia_xx">0.0</param>
+          <param name="payload_inertia_xy">0.0</param>
+          <param name="payload_inertia_xz">0.0</param>
+          <param name="payload_inertia_yy">0.0</param>
+          <param name="payload_inertia_yz">0.0</param>
+          <param name="payload_inertia_zz">0.0</param>
+        </xacro:if>
+      </hardware>
+      <joint name="waist">
+        <xacro:standard_interfaces />
+        <xacro:if value="${hardware == 'crcopen'}">
+          <xacro:crcopen_interfaces />
+          <param name="axis_idx">0</param>
+          <param name="ruckig_max_vel">${radians(110)}</param>
+          <param name="ruckig_max_acc">${radians(600)}</param>
+          <param name="ruckig_max_jrk">${radians(10000)}</param>
+          <!-- Motor constants -->
+          <param name="vr_TorqConst">1.0</param>            <!-- [Nm/A] -->
+          <param name="vr_TransmissionRatio">1.0</param>  <!-- [unitless] -->
+        </xacro:if>
+      </joint>
+      <joint name="shoulder">
+        <xacro:standard_interfaces />
+        <xacro:if value="${hardware == 'crcopen'}">
+          <xacro:crcopen_interfaces />
+          <param name="axis_idx">1</param>
+          <param name="ruckig_max_vel">${radians(110)}</param>
+          <param name="ruckig_max_acc">${radians(500)}</param>
+          <param name="ruckig_max_jrk">${radians(10000)}</param>
+          <!-- Motor constants -->
+          <param name="vr_TorqConst">1.0</param>            <!-- [Nm/A] -->
+          <param name="vr_TransmissionRatio">1.0</param>  <!-- [unitless] -->
+        </xacro:if>
+      </joint>
+      <joint name="elbow_active">
+        <xacro:standard_interfaces initial_position="${radians(-90)}" />
+        <xacro:if value="${hardware == 'crcopen'}">
+          <xacro:crcopen_interfaces />
+          <param name="axis_idx">2</param>
+          <param name="ruckig_max_vel">${radians(110)}</param>
+          <param name="ruckig_max_acc">${radians(850)}</param>
+          <param name="ruckig_max_jrk">${radians(15000)}</param>
+          <!-- Motor constants -->
+          <param name="vr_TorqConst">1.0</param>            <!-- [Nm/A] -->
+          <param name="vr_TransmissionRatio">1.0</param>  <!-- [Unitless] -->
+        </xacro:if>
+      </joint>
+      <joint name="forearm_roll">
+        <xacro:standard_interfaces />
+        <xacro:if value="${hardware == 'crcopen'}">
+          <xacro:crcopen_interfaces />
+          <param name="axis_idx">3</param>
+          <param name="ruckig_max_vel">${radians(190)}</param>
+          <param name="ruckig_max_acc">${radians(3400)}</param>
+          <param name="ruckig_max_jrk">${radians(90000)}</param>
+          <!-- Motor constants -->
+          <param name="vr_TorqConst">1.0</param>            <!-- [Nm/A] -->
+          <param name="vr_TransmissionRatio">1.0</param>   <!-- [Unitless] -->
+        </xacro:if>
+      </joint>
+      <joint name="wrist_angle">
+        <xacro:standard_interfaces />
+        <xacro:if value="${hardware == 'crcopen'}">
+          <xacro:crcopen_interfaces />
+          <param name="axis_idx">4</param>
+          <param name="ruckig_max_vel">${radians(190)}</param>
+          <param name="ruckig_max_acc">${radians(3300)}</param>
+          <param name="ruckig_max_jrk">${radians(90000)}</param>
+          <!-- Motor constants -->
+          <param name="vr_TorqConst">1.0</param>            <!-- [Nm/A] -->
+          <param name="vr_TransmissionRatio">1.0</param>   <!-- [Unitless] -->
+        </xacro:if>
+      </joint>
+      <joint name="wrist_rotate">
+        <xacro:standard_interfaces />
+        <xacro:if value="${hardware == 'crcopen'}">
+          <xacro:crcopen_interfaces />
+          <param name="axis_idx">5</param>
+          <param name="ruckig_max_vel">${radians(230)}</param>
+          <param name="ruckig_max_acc">${radians(4200)}</param>
+          <param name="ruckig_max_jrk">${radians(115000)}</param>
+          <!-- Motor constants -->
+          <param name="vr_TorqConst">1.0</param>            <!-- [Nm/A] -->
+          <param name="vr_TransmissionRatio">1.0</param>  <!-- [Unitless] -->
+        </xacro:if>
+      </joint>
+    </ros2_control>
   </xacro:macro>
-  <ros2_control name="comau_nj_130_2_6" type="system">
-    <hardware>
-        <plugin>crcopen_hardware/CRCOpenHardware</plugin>
-        <!-- Set IP addresses -->
-        <param name="lpc_addr">169.254.100.2</param>
-        <param name="crc_addr">169.254.100.1</param>
-        <!-- Set payload parameters -->
-        <param name="payload_mass">0.0</param>
-        <param name="payload_cog_x">0.0</param>
-        <param name="payload_cog_y">0.0</param>
-        <param name="payload_cog_z">0.0</param>
-        <param name="payload_inertia_xx">0.0</param>
-        <param name="payload_inertia_xy">0.0</param>
-        <param name="payload_inertia_xz">0.0</param>
-        <param name="payload_inertia_yy">0.0</param>
-        <param name="payload_inertia_yz">0.0</param>
-        <param name="payload_inertia_zz">0.0</param>
-    </hardware>
-    <joint name="waist">
-      <param name="axis_idx">0</param>
-      <param name="ruckig_max_vel">${radians(110)}</param>
-      <param name="ruckig_max_acc">${radians(600)}</param>
-      <param name="ruckig_max_jrk">${radians(10000)}</param>
-      <param name="vr_TorqConst">1.0</param>
-      <param name="vr_TransmissionRatio">1.0</param>
-      <xacro:all_command_and_state_interfaces />
-    </joint>
-    <joint name="shoulder">
-      <param name="axis_idx">1</param>
-      <param name="ruckig_max_vel">${radians(110)}</param>
-      <param name="ruckig_max_acc">${radians(500)}</param>
-      <param name="ruckig_max_jrk">${radians(10000)}</param>
-      <param name="vr_TorqConst">1.0</param>
-      <param name="vr_TransmissionRatio">1.0</param>
-      <xacro:all_command_and_state_interfaces />
-    </joint>
-    <joint name="elbow_active">
-      <param name="axis_idx">2</param>
-      <param name="ruckig_max_vel">${radians(110)}</param>
-      <param name="ruckig_max_acc">${radians(850)}</param>
-      <param name="ruckig_max_jrk">${radians(15000)}</param>
-      <param name="vr_TorqConst">1.0</param>
-      <param name="vr_TransmissionRatio">1.0</param>
-      <xacro:all_command_and_state_interfaces />
-    </joint>
-    <joint name="forearm_roll">
-      <param name="axis_idx">3</param>
-      <param name="ruckig_max_vel">${radians(190)}</param>
-      <param name="ruckig_max_acc">${radians(3400)}</param>
-      <param name="ruckig_max_jrk">${radians(90000)}</param>
-      <param name="vr_TorqConst">1.0</param>
-      <param name="vr_TransmissionRatio">1.0</param>
-      <xacro:all_command_and_state_interfaces />
-    </joint>
-    <joint name="wrist_angle">
-      <param name="axis_idx">4</param>
-      <param name="ruckig_max_vel">${radians(190)}</param>
-      <param name="ruckig_max_acc">${radians(3300)}</param>
-      <param name="ruckig_max_jrk">${radians(90000)}</param>
-      <param name="vr_TorqConst">1.0</param>
-      <param name="vr_TransmissionRatio">1.0</param>
-      <xacro:all_command_and_state_interfaces />
-    </joint>
-    <joint name="wrist_rotate">
-      <param name="axis_idx">5</param>
-      <param name="ruckig_max_vel">${radians(230)}</param>
-      <param name="ruckig_max_acc">${radians(4200)}</param>
-      <param name="ruckig_max_jrk">${radians(115000)}</param>
-      <param name="vr_TorqConst">1.0</param>
-      <param name="vr_TransmissionRatio">1.0</param>
-      <xacro:all_command_and_state_interfaces />
-    </joint>
-  </ros2_control>
 </robot>

File: comau_robots/comau_nj_130_2_6_description/urdf/nj_130_2_6_arm.urdf.xacro (robot description, xacro)
@@ -19,5 +19,5 @@
   <link name="base_link">
     <xacro:add_visual_and_collision link_name="link_0" xyz="0 0 0" rpy="0 0 0"/>
-    <!-- inertia: none because base is a fixed link -->
+    <!-- inertia, none because base is a fixed link -->
   </link>
   <link name="link_1_and_motors">
@@ -108,5 +108,5 @@
     <origin xyz="0.35 0 -0.499" rpy="${-pi/2} 0 ${pi}"/>
     <axis xyz="0 0 1"/>
-    <limit lower="${radians(-75)}" upper="${radians(60)}" velocity="${radians(110)}" effort="100000.0" />
+    <limit lower="${radians(-75)}" upper="${radians(95)}" velocity="${radians(110)}" effort="100000.0" />
   </joint>
   <joint name="elbow_active" type="revolute">

Commit message: [Jazzy] Update ROS 2 Jazzy support

File: comau_robots/comau_nj_130_2_6_description/urdf/nj_130_2_6.ros2_control.xacro (robot description, xacro)
@@ -1,83 +1,108 @@
 <?xml version="1.0"?>
 <robot xmlns:xacro="http://www.ros.org/wiki/xacro">
-  <xacro:macro name="all_command_and_state_interfaces">
-    <command_interface name="position"/>
-    <command_interface name="position_direct"/>
-    <command_interface name="velocity"/>
-    <command_interface name="acceleration"/>
-    <command_interface name="current"/>
-    <command_interface name="torque"/>
-    <state_interface name="position"/>
-    <state_interface name="velocity"/>
-    <state_interface name="acceleration"/>
-    <state_interface name="current"/>
-    <state_interface name="torque"/>
+  <xacro:include filename="$(find comau_nj_130_2_6_description)/urdf/helper_macros.urdf.xacro" />
+  <xacro:macro name="comau_nj_130_2_6_ros2_control" params="hardware:=crcopen">
+    <ros2_control name="comau_nj_130_2_6" type="system">
+      <hardware>
+        <xacro:if value="${hardware == 'mock'}">
+          <plugin>mock_components/GenericSystem</plugin>
+        </xacro:if>
+        <xacro:if value="${hardware == 'crcopen'}">
+          <plugin>crcopen_hardware/CRCOpenHardware</plugin>
+          <!-- Set IP addresses -->
+          <param name="lpc_addr">169.254.100.2</param>
+          <param name="crc_addr">169.254.100.1</param>
+          <!-- Set payload parameters -->
+          <param name="payload_mass">0.0</param>
+          <param name="payload_cog_x">0.0</param>
+          <param name="payload_cog_y">0.0</param>
+          <param name="payload_cog_z">0.0</param>
+          <param name="payload_inertia_xx">0.0</param>
+          <param name="payload_inertia_xy">0.0</param>
+          <param name="payload_inertia_xz">0.0</param>
+          <param name="payload_inertia_yy">0.0</param>
+          <param name="payload_inertia_yz">0.0</param>
+          <param name="payload_inertia_zz">0.0</param>
+        </xacro:if>
+      </hardware>
+      <joint name="waist">
+        <xacro:standard_interfaces />
+        <xacro:if value="${hardware == 'crcopen'}">
+          <xacro:crcopen_interfaces />
+          <param name="axis_idx">0</param>
+          <param name="ruckig_max_vel">${radians(110)}</param>
+          <param name="ruckig_max_acc">${radians(600)}</param>
+          <param name="ruckig_max_jrk">${radians(10000)}</param>
+          <!-- Motor constants -->
+          <param name="vr_TorqConst">1.0</param>            <!-- [Nm/A] -->
+          <param name="vr_TransmissionRatio">1.0</param>  <!-- [unitless] -->
+        </xacro:if>
+      </joint>
+      <joint name="shoulder">
+        <xacro:standard_interfaces />
+        <xacro:if value="${hardware == 'crcopen'}">
+          <xacro:crcopen_interfaces />
+          <param name="axis_idx">1</param>
+          <param name="ruckig_max_vel">${radians(110)}</param>
+          <param name="ruckig_max_acc">${radians(500)}</param>
+          <param name="ruckig_max_jrk">${radians(10000)}</param>
+          <!-- Motor constants -->
+          <param name="vr_TorqConst">1.0</param>            <!-- [Nm/A] -->
+          <param name="vr_TransmissionRatio">1.0</param>  <!-- [unitless] -->
+        </xacro:if>
+      </joint>
+      <joint name="elbow_active">
+        <xacro:standard_interfaces initial_position="${radians(-90)}" />
+        <xacro:if value="${hardware == 'crcopen'}">
+          <xacro:crcopen_interfaces />
+          <param name="axis_idx">2</param>
+          <param name="ruckig_max_vel">${radians(110)}</param>
+          <param name="ruckig_max_acc">${radians(850)}</param>
+          <param name="ruckig_max_jrk">${radians(15000)}</param>
+          <!-- Motor constants -->
+          <param name="vr_TorqConst">1.0</param>            <!-- [Nm/A] -->
+          <param name="vr_TransmissionRatio">1.0</param>  <!-- [Unitless] -->
+        </xacro:if>
+      </joint>
+      <joint name="forearm_roll">
+        <xacro:standard_interfaces />
+        <xacro:if value="${hardware == 'crcopen'}">
+          <xacro:crcopen_interfaces />
+          <param name="axis_idx">3</param>
+          <param name="ruckig_max_vel">${radians(190)}</param>
+          <param name="ruckig_max_acc">${radians(3400)}</param>
+          <param name="ruckig_max_jrk">${radians(90000)}</param>
+          <!-- Motor constants -->
+          <param name="vr_TorqConst">1.0</param>            <!-- [Nm/A] -->
+          <param name="vr_TransmissionRatio">1.0</param>   <!-- [Unitless] -->
+        </xacro:if>
+      </joint>
+      <joint name="wrist_angle">
+        <xacro:standard_interfaces />
+        <xacro:if value="${hardware == 'crcopen'}">
+          <xacro:crcopen_interfaces />
+          <param name="axis_idx">4</param>
+          <param name="ruckig_max_vel">${radians(190)}</param>
+          <param name="ruckig_max_acc">${radians(3300)}</param>
+          <param name="ruckig_max_jrk">${radians(90000)}</param>
+          <!-- Motor constants -->
+          <param name="vr_TorqConst">1.0</param>            <!-- [Nm/A] -->
+          <param name="vr_TransmissionRatio">1.0</param>   <!-- [Unitless] -->
+        </xacro:if>
+      </joint>
+      <joint name="wrist_rotate">
+        <xacro:standard_interfaces />
+        <xacro:if value="${hardware == 'crcopen'}">
+          <xacro:crcopen_interfaces />
+          <param name="axis_idx">5</param>
+          <param name="ruckig_max_vel">${radians(230)}</param>
+          <param name="ruckig_max_acc">${radians(4200)}</param>
+          <param name="ruckig_max_jrk">${radians(115000)}</param>
+          <!-- Motor constants -->
+          <param name="vr_TorqConst">1.0</param>            <!-- [Nm/A] -->
+          <param name="vr_TransmissionRatio">1.0</param>  <!-- [Unitless] -->
+        </xacro:if>
+      </joint>
+    </ros2_control>
   </xacro:macro>
-  <ros2_control name="comau_nj_130_2_6" type="system">
-    <hardware>
-        <plugin>crcopen_hardware/CRCOpenHardware</plugin>
-        <!-- Set IP addresses -->
-        <param name="lpc_addr">169.254.100.2</param>
-        <param name="crc_addr">169.254.100.1</param>
-        <!-- Set payload parameters -->
-        <param name="payload_mass">0.0</param>
-        <param name="payload_cog_x">0.0</param>
-        <param name="payload_cog_y">0.0</param>
-        <param name="payload_cog_z">0.0</param>
-        <param name="payload_inertia_xx">0.0</param>
-        <param name="payload_inertia_xy">0.0</param>
-        <param name="payload_inertia_xz">0.0</param>
-        <param name="payload_inertia_yy">0.0</param>
-        <param name="payload_inertia_yz">0.0</param>
-        <param name="payload_inertia_zz">0.0</param>
-    </hardware>
-    <joint name="waist">
-      <param name="axis_idx">0</param>
-      <param name="ruckig_max_vel">${radians(110)}</param>
-      <param name="ruckig_max_acc">${radians(600)}</param>
-      <param name="ruckig_max_jrk">${radians(10000)}</param>
-      <param name="vr_TorqConst">1.0</param>
-      <xacro:all_command_and_state_interfaces />
-    </joint>
-    <joint name="shoulder">
-      <param name="axis_idx">1</param>
-      <param name="ruckig_max_vel">${radians(110)}</param>
-      <param name="ruckig_max_acc">${radians(500)}</param>
-      <param name="ruckig_max_jrk">${radians(10000)}</param>
-      <param name="vr_TorqConst">1.0</param>
-      <xacro:all_command_and_state_interfaces />
-    </joint>
-    <joint name="elbow_active">
-      <param name="axis_idx">2</param>
-      <param name="ruckig_max_vel">${radians(110)}</param>
-      <param name="ruckig_max_acc">${radians(850)}</param>
-      <param name="ruckig_max_jrk">${radians(15000)}</param>
-      <param name="vr_TorqConst">1.0</param>
-      <xacro:all_command_and_state_interfaces />
-    </joint>
-    <joint name="forearm_roll">
-      <param name="axis_idx">3</param>
-      <param name="ruckig_max_vel">${radians(190)}</param>
-      <param name="ruckig_max_acc">${radians(3400)}</param>
-      <param name="ruckig_max_jrk">${radians(90000)}</param>
-      <param name="vr_TorqConst">1.0</param>
-      <xacro:all_command_and_state_interfaces />
-    </joint>
-    <joint name="wrist_angle">
-      <param name="axis_idx">4</param>
-      <param name="ruckig_max_vel">${radians(190)}</param>
-      <param name="ruckig_max_acc">${radians(3300)}</param>
-      <param name="ruckig_max_jrk">${radians(90000)}</param>
-      <param name="vr_TorqConst">1.0</param>
-      <xacro:all_command_and_state_interfaces />
-    </joint>
-    <joint name="wrist_rotate">
-      <param name="axis_idx">5</param>
-      <param name="ruckig_max_vel">${radians(230)}</param>
-      <param name="ruckig_max_acc">${radians(4200)}</param>
-      <param name="ruckig_max_jrk">${radians(115000)}</param>
-      <param name="vr_TorqConst">1.0</param>
-      <xacro:all_command_and_state_interfaces />
-    </joint>
-  </ros2_control>
 </robot>
